File: PCB/IR_to_USB.sch (KiCad schematic (older format))
At the start: 5 parts, among them U1 STM32F070CBT6

Commit message: PCB in progress
Signed-off-by: denis-m-tyurin <denis.m.turin@gmail.com>
Parts:
- added C1, C4, C8: 100 nF, Capacitors_SMD:C_1206_HandSoldering, symbol C
- added C3: 330 nF, Capacitors_SMD:C_1206_HandSoldering, symbol C
- added D1: LED_RGB, LEDs:LED_RGB_PLLC-6, symbol LED_RGB
- added JP1: JUMPER, Buttons_Switches_ThroughHole:SW_DIP_x1_Slide, symbol JUMPER
- added P1: CONN_01X06, Connect:PINHEAD1-6, symbol CONN_01X06
- added P2: USB_OTG, Connect:USB_Mini-B, symbol USB_OTG
- added R1, R2: 10K, Resistors_SMD:R_1206_HandSoldering, symbol R
- added R3: 62, Resistors_SMD:R_1206_HandSoldering, symbol R
- added R4, R5: 5, Resistors_SMD:R_1206_HandSoldering, symbol R
- added R6, R7: 33, Resistors_SMD:R_1206_HandSoldering, symbol R
- added SW1: SW_PUSH, Buttons_Switches_ThroughHole:SW_PUSH-12mm, symbol SW_PUSH
- added U1: L78L, TO_SOT_Packages_THT:TO-92_Inline_Narrow_Oval, symbol L78L
- added U3: TSOP48, TO_SOT_Packages_THT:TO-220_Neutral123_Horizontal_LargePads, symbol TSOP48
- added X1: CRYSTAL_SMD, Footprint_lib:CSTCE_G_Murata_Resonator, symbol CRYSTAL_SMD
- C2: renamed from C4; footprint Capacitors_SMD:C_1206 -> Capacitors_SMD:C_1206_HandSoldering
- C5: renamed from C1; footprint Capacitors_SMD:C_1206 -> Capacitors_SMD:C_1206_HandSoldering
- C6: renamed from C2; footprint Capacitors_SMD:C_1206 -> Capacitors_SMD:C_1206_HandSoldering
- C7: renamed from C3; footprint Capacitors_SMD:C_1206 -> Capacitors_SMD:C_1206_HandSoldering
- renumbered U1 to U2
Connections:
- net +3V3: now also C2.2, U2.1 (VBAT), U2.36 (VDD), C1.1, C8.1, P1.2 (P2), R1.1, R2.1, U1.1 (OUT), U3.3 (Vs)
- net Earth: now also C1.2, C3.2, C4.1, C8.2, D1.1 (RC), D1.2 (GC), D1.3 (BC), JP1.1, P1.1 (P1), P1.5 (P5), P2.5 (GND), SW1.2, U1.2 (GND), U3.2 (GND), X1.2
- net at U2.11 (ADC1_IN1/TIM2_CH2/PA1): now also R3.1
- net at U2.12 (ADC1_IN2/TIM2_CH3/PA2): now also R4.1
- net at U2.13 (ADC1_IN3/TIM2_CH4/PA3): now also R5.1
- net at U2.16 (SPI1_MISO/I2S1_MCK/TIM3_CH1/TIM1_BKIN/ADC_IN6/TIM16_CH1/EVENTOUT/PA6): now also U3.1 (OUT)
- net at U2.32 (USART1_CTS/TIM1_CH4/EVENTOUT/PA11): now also R6.2
- net at U2.33 (USART1_RTS/TIM1_ETR/EVENTOUT/PA12): now also R7.2
- net at U2.34 (IR_OUT/SWDAT/PA13): now also P1.3 (P3)
- net at U2.37 (SWCLK/PA14): now also P1.4 (P4)
- net at U2.44 (BOOT0): now also JP1.2, R1.2
- net at U2.5 (PF0/OSC_IN): now also X1.3 (case)
- net at U2.6 (PF1/OSC_OUT): now also X1.1
- net at U2.7 (~NRST): now also C4.2, P1.6 (P6), R2.2, SW1.1
- new net: P2.2 (D-), R6.1
- new net: P2.3 (D+), R7.1
- new net: D1.4 (BA), R5.2
- new net: D1.5 (GA), R4.2
- new net: D1.6 (RA), R3.2
- new net +5V: C3.1, P2.1 (VCC), U1.3 (IN)
- no-connect marks 0 -> 30

Commit message: Rework PCB: changed RGB led type, removed reset button, etc.
Signed-off-by: denis-m-tyurin <denis.m.turin@gmail.com>
Parts:
- removed D1: LED_RGB, LEDs:LED_RGB_PLLC-6, symbol LED_RGB
- removed R2: 10K, Resistors_SMD:R_1206_HandSoldering, symbol R
- removed SW1: SW_PUSH, Buttons_Switches_ThroughHole:SW_PUSH-12mm, symbol SW_PUSH
- added D1: LED_RABG, LEDs:LED-RGB-5MM_Common_Cathode, symbol LED_RABG
- U1: footprint TO_SOT_Packages_THT:TO-92_Inline_Narrow_Oval -> TO_SOT_Packages_THT:TO-220_Neutral123_PadsOnly
Connections:
- net +3V3: now also D1.2 (COMMON_ANODE)
- net at R5.2: now also D1.4 (GREEN_CATHODE)
- net at R4.2: now also D1.3 (BLUE_CATHODE)
- net at R3.2: now also D1.1 (RED_CATHODE)
Changed lines of the file:
@@
 	4650 1500 4650 1400
 $Comp
-L Earth #PWR01
+L Earth #PWR9
 U 1 1 561283CE
 P 4100 5450
-F 0 "#PWR01" H 4100 5200 50  0001 C CNN
+F 0 "#PWR9" H 4100 5200 50  0001 C CNN
 F 1 "Earth" H 4100 5300 50  0001 C CNN
 F 2 "" H 4100 5450 60  0000 C CNN
@@
 $EndComp
 $Comp
-L Earth #PWR02
+L Earth #PWR10
 U 1 1 561283F2
 P 4250 5450
-F 0 "#PWR02" H 4250 5200 50  0001 C CNN
+F 0 "#PWR10" H 4250 5200 50  0001 C CNN
 F 1 "Earth" H 4250 5300 50  0001 C CNN
 F 2 "" H 4250 5450 60  0000 C CNN
@@
 $EndComp
 $Comp
-L Earth #PWR03
+L Earth #PWR11
 U 1 1 56128809
 P 4550 5450
-F 0 "#PWR03" H 4550 5200 50  0001 C CNN
+F 0 "#PWR11" H 4550 5200 50  0001 C CNN
 F 1 "Earth" H 4550 5300 50  0001 C CNN
 F 2 "" H 4550 5450 60  0000 C CNN
@@
 	2100 3700 1800 3700
 $Comp
-L Earth #PWR04
+L Earth #PWR5
 U 1 1 56128D3D
 P 1800 3700
-F 0 "#PWR04" H 1800 3450 50  0001 C CNN
+F 0 "#PWR5" H 1800 3450 50  0001 C CNN
 F 1 "Earth" H 1800 3550 50  0001 C CNN
 F 2 "" H 1800 3700 60  0000 C CNN
@@
 Connection ~ 2050 3700
 $Comp
-L Earth #PWR05
+L Earth #PWR8
 U 1 1 56128FA8
 P 3500 950
-F 0 "#PWR05" H 3500 700 50  0001 C CNN
+F 0 "#PWR8" H 3500 700 50  0001 C CNN
 F 1 "Earth" H 3500 800 50  0001 C CNN
 F 2 "" H 3500 950 60  0000 C CNN
@@
 	3750 950  3500 950
 $Comp
-L Earth #PWR06
+L Earth #PWR12
 U 1 1 56128FFD
 P 4650 750
-F 0 "#PWR06" H 4650 500 50  0001 C CNN
+F 0 "#PWR12" H 4650 500 50  0001 C CNN
 F 1 "Earth" H 4650 600 50  0001 C CNN
 F 2 "" H 4650 750 60  0000 C CNN
@@
 	4400 750  4650 750
 $Comp
-L Earth #PWR07
+L Earth #PWR13
 U 1 1 5612904C
 P 4950 1100
-F 0 "#PWR07" H 4950 850 50  0001 C CNN
+F 0 "#PWR13" H 4950 850 50  0001 C CNN
 F 1 "Earth" H 4950 950 50  0001 C CNN
 F 2 "" H 4950 1100 60  0000 C CNN
@@
 	4800 1100 4950 1100
 $Comp
-L +3.3V #PWR08
+L +3.3V #PWR14
 U 1 1 5612923E
 P 5550 750
-F 0 "#PWR08" H 5550 600 50  0001 C CNN
+F 0 "#PWR14" H 5550 600 50  0001 C CNN
 F 1 "+3.3V" H 5550 890 50  0000 C CNN
 F 2 "" H 5550 750 60  0000 C CNN
@@
 Connection ~ 4550 1400
 $Comp
-L Earth #PWR09
+L Earth #PWR2
 U 1 1 561622CD
 P 1000 2000
-F 0 "#PWR09" H 1000 1750 50  0001 C CNN
+F 0 "#PWR2" H 1000 1750 50  0001 C CNN
 F 1 "Earth" H 1000 1850 50  0001 C CNN
 F 2 "" H 1000 2000 60  0000 C CNN
@@
 $EndComp
 $Comp
-L Earth #PWR010
+L Earth #PWR7
 U 1 1 561643AF
 P 2850 1200
-F 0 "#PWR010" H 2850 950 50  0001 C CNN
+F 0 "#PWR7" H 2850 950 50  0001 C CNN
 F 1 "Earth" H 2850 1050 50  0001 C CNN
 F 2 "" H 2850 1200 60  0000 C CNN
@@
 	2600 1200 2600 1100
 Wire Wire Line
-	2600 1100 2950 1100
-Wire Wire Line
 	2850 1100 2850 1200
 Wire Wire Line
@@
 Wire Wire Line
 	2100 1500 2600 1500
-$Comp
-L SW_PUSH SW1
-U 1 1 5616461E
-P 2650 950
-F 0 "SW1" H 2800 1060 50  0000 C CNN
-F 1 "SW_PUSH" H 2650 870 50  0000 C CNN
-F 2 "Buttons_Switches_ThroughHole:SW_PUSH-12mm" H 2650 950 60  0000 C CNN
-F 3 "" H 2650 950 60  0000 C CNN
-	1    2650 950
-	1    0    0    -1
-$EndComp
-Wire Wire Line
-	2950 1100 2950 950
-Connection ~ 2850 1100
-Wire Wire Line
-	2350 1500 2350 950
 Connection ~ 2550 1500
-$Comp
-L R R2
-U 1 1 561647AD
-P 2250 1200
-F 0 "R2" V 2330 1200 50  0000 C CNN
-F 1 "10K" V 2250 1200 50  0000 C CNN
-F 2 "Resistors_SMD:R_1206_HandSoldering" V 2180 1200 30  0000 C CNN
-F 3 "" H 2250 1200 30  0000 C CNN
-	1    2250 1200
-	1    0    0    -1
-$EndComp
-Wire Wire Line
-	2250 1500 2250 1350
-Connection ~ 2350 1500
-Wire Wire Line
-	2250 1050 2250 600
-Connection ~ 2250 600
 Connection ~ 5350 900
 $Comp
-L Earth #PWR011
+L Earth #PWR16
 U 1 1 561653D5
 P 8500 1500
-F 0 "#PWR011" H 8500 1250 50  0001 C CNN
+F 0 "#PWR16" H 8500 1250 50  0001 C CNN
 F 1 "Earth" H 8500 1350 50  0001 C CNN
 F 2 "" H 8500 1500 60  0000 C CNN
@@
 Wire Wire Line
 	7050 550  7050 1700
-Connection ~ 2250 1500
 $Comp
 L USB_OTG P2
@@
 $EndComp
 $Comp
-L +5V #PWR012
+L +5V #PWR15
 U 1 1 56167140
 P 8300 2400
-F 0 "#PWR012" H 8300 2250 50  0001 C CNN
+F 0 "#PWR15" H 8300 2250 50  0001 C CNN
 F 1 "+5V" H 8300 2540 50  0000 C CNN
 F 2 "" H 8300 2400 60  0000 C CNN
@@
 	8300 2600 8300 2400
 $Comp
-L Earth #PWR013
+L Earth #PWR19
 U 1 1 561671CD
 P 9600 2700
-F 0 "#PWR013" H 9600 2450 50  0001 C CNN
+F 0 "#PWR19" H 9600 2450 50  0001 C CNN
 F 1 "Earth" H 9600 2550 50  0001 C CNN
 F 2 "" H 9600 2700 60  0000 C CNN
@@
 $EndComp
 $Comp
-L Earth #PWR014
+L Earth #PWR1
 U 1 1 5616909A
 P 750 3850
-F 0 "#PWR014" H 750 3600 50  0001 C CNN
+F 0 "#PWR1" H 750 3600 50  0001 C CNN
 F 1 "Earth" H 750 3700 50  0001 C CNN
 F 2 "" H 750 3850 60  0000 C CNN
@@
 Wire Wire Line
 	1050 3450 1050 3750
-$Comp
-L LED_RGB D1
-U 1 1 5616A801
-P 7800 2550
-F 0 "D1" H 7800 2975 50  0000 C CNN
-F 1 "LED_RGB" H 7800 2900 50  0000 C CNN
-F 2 "LEDs:LED_RGB_PLLC-6" H 7800 2500 50  0000 C CNN
-F 3 "" H 7800 2500 50  0000 C CNN
-	1    7800 2550
-	-1   0    0    1
-$EndComp
 $Comp
 L R R5
@@
 $EndComp
 Wire Wire Line
-	7600 2350 7450 2350
-Wire Wire Line
-	7450 2350 7450 2450
-Wire Wire Line
-	7450 2450 7350 2450
-Wire Wire Line
-	7350 2450 7350 2400
-Wire Wire Line
-	7600 2550 7200 2550
-Wire Wire Line
-	7200 2550 7200 2400
-Wire Wire Line
-	7600 2750 7050 2750
+	7350 2400 7350 2550
+Wire Wire Line
+	7200 2400 7200 2650
 Wire Wire Line
 	7050 2750 7050 2400
@@
 Wire Wire Line
 	7350 2100 7350 1950
-$Comp
-L Earth #PWR015
-U 1 1 5616CF4B
-P 8150 2850
-F 0 "#PWR015" H 8150 2600 50  0001 C CNN
-F 1 "Earth" H 8150 2700 50  0001 C CNN
-F 2 "" H 8150 2850 60  0000 C CNN
-F 3 "" H 8150 2850 60  0000 C CNN
-	1    8150 2850
-	1    0    0    -1
-$EndComp
-Wire Wire Line
-	8150 2850 8150 2350
-Wire Wire Line
-	8150 2350 8000 2350
-Wire Wire Line
-	8000 2550 8150 2550
-Connection ~ 8150 2550
-Wire Wire Line
-	8000 2750 8150 2750
-Connection ~ 8150 2750
 NoConn ~ 9150 2600
 NoConn ~ 9450 2200
 NoConn ~ 10200 1550
 $Comp
-L +3.3V #PWR016
+L +3.3V #PWR3
 U 1 1 561B7D1A
 P 1100 5850
-F 0 "#PWR016" H 1100 5700 50  0001 C CNN
+F 0 "#PWR3" H 1100 5700 50  0001 C CNN
 F 1 "+3.3V" H 1100 5990 50  0000 C CNN
 F 2 "" H 1100 5850 60  0000 C CNN
@@
 $EndComp
 $Comp
-L Earth #PWR017
+L Earth #PWR4
 U 1 1 561B7EF6
 P 1700 6500
-F 0 "#PWR017" H 1700 6250 50  0001 C CNN
+F 0 "#PWR4" H 1700 6250 50  0001 C CNN
 F 1 "Earth" H 1700 6350 50  0001 C CNN
 F 2 "" H 1700 6500 60  0000 C CNN
@@
 $EndComp
 $Comp
-L Earth #PWR018
+L Earth #PWR17
 U 1 1 561BBA07
 P 8600 5550
-F 0 "#PWR018" H 8600 5300 50  0001 C CNN
+F 0 "#PWR17" H 8600 5300 50  0001 C CNN
 F 1 "Earth" H 8600 5400 50  0001 C CNN
 F 2 "" H 8600 5550 60  0000 C CNN
@@
 $EndComp
 $Comp
-L +3.3V #PWR019
+L +3.3V #PWR18
 U 1 1 561BC299
 P 9400 4650
-F 0 "#PWR019" H 9400 4500 50  0001 C CNN
+F 0 "#PWR18" H 9400 4500 50  0001 C CNN
 F 1 "+3.3V" H 9400 4790 50  0000 C CNN
 F 2 "" H 9400 4650 60  0000 C CNN
@@
 F 0 "U1" H 1500 6300 40  0000 C CNN
 F 1 "L78L" H 1700 6300 40  0000 L CNN
-F 2 "TO_SOT_Packages_THT:TO-92_Inline_Narrow_Oval" H 1700 6200 30  0000 C CIN
+F 2 "TO_SOT_Packages_THT:TO-220_Neutral123_PadsOnly" H 1700 6200 30  0000 C CIN
 F 3 "" H 1700 6100 60  0000 C CNN
 	1    1700 6100
@@
 Connection ~ 2300 2300
 $Comp
-L Earth #PWR020
+L Earth #PWR6
 U 1 1 561C7554
 P 2300 2700
-F 0 "#PWR020" H 2300 2450 50  0001 C CNN
+F 0 "#PWR6" H 2300 2450 50  0001 C CNN
 F 1 "Earth" H 2300 2550 50  0001 C CNN
 F 2 "" H 2300 2700 60  0000 C CNN
@@
 Wire Wire Line
 	6600 2150 5950 2150
+Wire Wire Line
+	2600 1100 2850 1100
+Wire Wire Line
+	7200 2650 7550 2650
+Wire Wire Line
+	7450 2350 7600 2350
+Wire Wire Line
+	7350 2550 7600 2550
+$Comp
+L LED_RABG D1
+U 1 1 5624F99B
+P 7900 2550
+F 0 "D1" H 7975 2900 50  0000 C CNN
+F 1 "LED_RABG" H 7925 2200 50  0000 C CNN
+F 2 "LEDs:LED-RGB-5MM_Common_Cathode" H 7850 2500 50  0000 C CNN
+F 3 "" H 7850 2500 50  0000 C CNN
+	1    7900 2550
+	1    0    0    -1
+$EndComp
+Wire Wire Line
+	8200 2550 8200 2100
+Wire Wire Line
+	8200 2100 7550 2100
+Wire Wire Line
+	7550 2100 7550 1400
+Connection ~ 7550 1400
+Wire Wire Line
+	7550 2650 7550 2750
+Wire Wire Line
+	7550 2750 7600 2750
+Wire Wire Line
+	7050 2750 7450 2750
+Wire Wire Line
+	7450 2750 7450 2350
 $EndSCHEMATC

Commit message: Reworked PCB to double layers
Signed-off-by: denis-m-tyurin <denis.m.turin@gmail.com>
Parts:
- added P3: CONN_01X02, Footprint_lib:PINHEAD1-2_withoutSilk, symbol CONN_01X02
- added P4: CONN_01X01, Connect:PINTST, symbol CONN_01X01
- C1, C2, C3, C4, C5, C6, C7, C8: footprint Capacitors_SMD:C_1206_HandSoldering -> Footprint_lib:C_1206_HandSoldering_withoutSilk
- D1: footprint LEDs:LED-RGB-5MM_Common_Cathode -> Footprint_lib:LED-RGB-5MM_Common_Cathode_DENIS
- JP1: footprint Buttons_Switches_ThroughHole:SW_DIP_x1_Slide -> Footprint_lib:SW_DIP_x1_Slide_DENIS
- P1: footprint Connect:PINHEAD1-6 -> Footprint_lib:PINHEAD1-6_DENIS
- R1, R3, R4, R5, R6, R7: footprint Resistors_SMD:R_1206_HandSoldering -> Footprint_lib:R_1206_HandSoldering_withoutSilk
- U2: symbol STM32F050C6 -> STM32F050C6-RESCUE-IR_to_USB
- U3: footprint TO_SOT_Packages_THT:TO-220_Neutral123_Horizontal_LargePads -> Footprint_lib:TO-220_Neutral123_Horizontal_LargePads_withoutSilk
- X1: footprint Footprint_lib:CSTCE_G_Murata_Resonator -> Footprint_lib:CSTCE_G_Murata_Resonator_withoutSilk
Connections:
- net at U2.14 (SPI1_NSS/I2S1_WS/ADC_IN4/TIM14_CH1/PA4): now also P3.1 (P1)
- net at U2.15 (SPI1_SCK/I2S1_CK/TIM2_CH1_ETR/ADC1_IN5/PA5): now also R6.2, U2.32 (USART1_CTS/TIM1_CH4/EVENTOUT/PA11), P3.2 (P2)
- net at U2.41 (SPI1_MOSI/I2S1_SD/I2C1_SMBA/TIM16_BKIN/TIM3_CH2/PB5): now also P4.1 (P1)
- no-connect marks 30 -> 27
